File: PCB/ahe_v1_0.brd (EAGLE design)
At the start: 61 x 61 mm, 41 parts, among them CN3 1X4-3.5MM, CN4 1X4-3.5MM, IC1 MS560702BA03-50, IC2 MCP73871-1CCI_ML, IC3 ESP32-S2-WROOM-I_M22S2H3200UH3, J1 USB3075-30-A, Q1 TSM200N03DPQ33_RGG

Commit message: Fixed known BMS issues
Connections:
- removed net N$5: IC2.1
- new net VBAT_OUT: C4.1, IC2.1, IC2.20, PS1.1, PS1.3
- net GND: now also IC2.21
- net V_BAT: no longer C4.1, PS1.1, PS1.3
Routing:
- net VBAT_OUT: track 0.00 -> 25.9 mm, vias 0 -> 2
- net V_BAT: track 78.3 -> 63.7 mm
- net VCC: track 108.9 -> 104.9 mm
