File: PCB/aprs_gps_v2/aprs_v2.sch (EAGLE design)
At the start: 17 parts, among them X1 BU-SMA-V

Commit message: fix VCC and Vin
Parts:
- added JP4: (no value), pinhead:PINHD-1X2
Connections:
- net GND: now also JP4.1
- net VCC: now also JP4.2, U$2.RAW
Changed lines of the file:
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@@
 <setting verticaltext="up"/>
 </settings>
-<grid distance="0.05" unitdist="inch" unit="inch" style="lines" multiple="1" display="yes" altdistance="0.01" altunitdist="inch" altunit="inch"/>
+<grid distance="0.1" unitdist="inch" unit="inch" style="lines" multiple="1" display="no" altdistance="0.01" altunitdist="inch" altunit="inch"/>
 <layers>
 <layer number="1" name="Top" color="4" fill="1" visible="no" active="no"/>
@@
 <part name="JP2" library="pinhead" library_urn="urn:adsk.eagle:library:325" deviceset="PINHD-1X4" device="" package3d_urn="urn:adsk.eagle:package:22407/2"/>
 <part name="JP3" library="pinhead" library_urn="urn:adsk.eagle:library:325" deviceset="PINHD-1X4" device="" package3d_urn="urn:adsk.eagle:package:22407/2"/>
+<part name="JP4" library="pinhead" library_urn="urn:adsk.eagle:library:325" deviceset="PINHD-1X2" device="" package3d_urn="urn:adsk.eagle:package:22435/2"/>
 </parts>
 <sheets>
@@
 <attribute name="NAME" x="96.52" y="14.605" size="1.778" layer="95"/>
 <attribute name="VALUE" x="96.52" y="-1.27" size="1.778" layer="96"/>
+</instance>
+<instance part="JP4" gate="G$1" x="-31.75" y="-1.27" smashed="yes" rot="R180">
+<attribute name="NAME" x="-25.4" y="-6.985" size="1.778" layer="95" rot="R180"/>
+<attribute name="VALUE" x="-25.4" y="3.81" size="1.778" layer="96" rot="R180"/>
 </instance>
 </instances>
@@
 <wire x1="92.71" y1="3.81" x2="92.71" y2="-8.89" width="0.1524" layer="91"/>
 <junction x="92.71" y="-8.89"/>
+<pinref part="JP4" gate="G$1" pin="1"/>
+<wire x1="-29.21" y1="-3.81" x2="-21.59" y2="-3.81" width="0.1524" layer="91"/>
+<wire x1="-21.59" y1="-3.81" x2="-21.59" y2="-5.08" width="0.1524" layer="91"/>
+<wire x1="-21.59" y1="-5.08" x2="-15.24" y2="-5.08" width="0.1524" layer="91"/>
+<junction x="-15.24" y="-5.08"/>
 </segment>
 </net>
@@
 <wire x1="34.29" y1="13.97" x2="30.48" y2="13.97" width="0.1524" layer="91"/>
 <wire x1="30.48" y1="13.97" x2="30.48" y2="11.43" width="0.1524" layer="91"/>
-<wire x1="30.48" y1="11.43" x2="30.48" y2="-6.35" width="0.1524" layer="91"/>
+<wire x1="30.48" y1="11.43" x2="30.48" y2="7.62" width="0.1524" layer="91"/>
+<wire x1="30.48" y1="7.62" x2="30.48" y2="-6.35" width="0.1524" layer="91"/>
 <wire x1="30.48" y1="-6.35" x2="71.12" y2="-6.35" width="0.1524" layer="91"/>
 <wire x1="71.12" y1="-6.35" x2="71.12" y2="-17.78" width="0.1524" layer="91"/>
@@
 <junction x="30.48" y="11.43"/>
 <wire x1="30.48" y1="11.43" x2="-8.89" y2="11.43" width="0.1524" layer="91"/>
-<wire x1="-8.89" y1="11.43" x2="-8.89" y2="2.54" width="0.1524" layer="91"/>
+<wire x1="-8.89" y1="11.43" x2="-8.89" y2="6.35" width="0.1524" layer="91"/>
 <pinref part="JP2" gate="A" pin="4"/>
+<wire x1="-8.89" y1="6.35" x2="-8.89" y2="2.54" width="0.1524" layer="91"/>
 <wire x1="-8.89" y1="2.54" x2="-15.24" y2="2.54" width="0.1524" layer="91"/>
+<pinref part="JP4" gate="G$1" pin="2"/>
+<wire x1="-29.21" y1="-1.27" x2="-22.86" y2="-1.27" width="0.1524" layer="91"/>
+<wire x1="-22.86" y1="-1.27" x2="-22.86" y2="6.35" width="0.1524" layer="91"/>
+<wire x1="-22.86" y1="6.35" x2="-8.89" y2="6.35" width="0.1524" layer="91"/>
+<junction x="-8.89" y="6.35"/>
+<pinref part="U$2" gate="G$1" pin="RAW"/>
+<wire x1="30.48" y1="7.62" x2="34.29" y2="7.62" width="0.1524" layer="91"/>
+<wire x1="34.29" y1="7.62" x2="34.29" y2="6.35" width="0.1524" layer="91"/>
+<junction x="30.48" y="7.62"/>
 </segment>
 <segment>
