File: GMP_SCH.brd (EAGLE design)
At the start: 68.1 x 65.3 mm, 24 parts, among them CN1 1X4-3.5MM, CN2 1X4-3.5MM, IC1 MS560702BA03-50, Q1 TSM200N03DPQ33_RGG

Commit message: Add files via upload
V1.2, Test ready, Added decals
Parts:
- moved JP3 6.10 mm to (10.5, 48.4)
Connections:
- net GND renamed BARE
Routing:
- net SERIAL_ESP_RX: track 11.9 -> 7.47 mm
- net SERIAL_ESP_TX: track 13.6 -> 9.79 mm
Other:
- board text added: "Matthew 10:28"
- board text added: "Not because it is easy but because it is hard"
- board text added: "V1.2"
Changed lines of the file:
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@@
 <wire x1="66.04" y1="65.278" x2="66.04" y2="0" width="0.3048" layer="20"/>
 <wire x1="66.04" y1="0" x2="-2.032" y2="0" width="0.3048" layer="20"/>
+<text x="11.684" y="60.706" size="1.778" layer="42" rot="MR0" grouprefs="BOARD">Piatt Labs</text>
+<text x="62.992" y="60.706" size="1.778" layer="42" rot="MR0">V1.2</text>
+<text x="13.716" y="49.022" size="1.778" layer="42" rot="MR0">Not because
+it is easy
+but because
+it is hard</text>
+<text x="64.262" y="6.858" size="1.778" layer="42" rot="MR315">Matthew
+10:28</text>
 </plain>
 <attributes>
@@
 <attribute name="VALUE" x="39.37" y="10.8204" size="1.27" layer="27" rot="R180"/>
 </element>
-<element name="JP3" library="pinhead" library_urn="urn:adsk.eagle:library:325" package="1X04/90" package3d_urn="urn:adsk.eagle:package:22404/2" value="" x="4.3942" y="48.133" smashed="yes" rot="R50" grouprefs="BOARD">
-<attribute name="NAME" x="3.63929375" y="41.306025" size="1.27" layer="25" ratio="10" rot="R140"/>
-<attribute name="POPULARITY" value="9" x="36.09683125" y="46.399334375" size="1.778" layer="27" rot="R50" display="off"/>
-<attribute name="VALUE" x="12.2891375" y="50.62661875" size="1.27" layer="27" rot="R140"/>
+<element name="JP3" library="pinhead" library_urn="urn:adsk.eagle:library:325" package="1X04/90" package3d_urn="urn:adsk.eagle:package:22404/2" value="" x="10.4902" y="48.387" smashed="yes" rot="R50" grouprefs="BOARD">
+<attribute name="NAME" x="9.73529375" y="41.560025" size="1.27" layer="25" ratio="10" rot="R140"/>
+<attribute name="POPULARITY" value="9" x="42.19283125" y="46.653334375" size="1.778" layer="27" rot="R50" display="off"/>
+<attribute name="VALUE" x="18.3851375" y="50.88061875" size="1.27" layer="27" rot="R140"/>
 </element>
 <element name="LED1" library="led" library_urn="urn:adsk.eagle:library:259" package="LED3MM" package3d_urn="urn:adsk.eagle:package:15797/1" value="TLLG4400" x="53.6702" y="15.7226" smashed="yes" grouprefs="BOARD">
@@
 <contactref element="JP3" pad="4"/>
 </signal>
-<signal name="GND">
+<signal name="BARE">
 <contactref element="C4" pad="2"/>
 <contactref element="C5" pad="2"/>
@@
 <contactref element="SV1" pad="7"/>
 <polygon width="0.1524" layer="16" spacing="0.3556">
-<vertex x="-1.3462" y="0.4318"/>
-<vertex x="-1.3462" y="65.0748"/>
-<vertex x="65.6844" y="65.0748"/>
+<vertex x="-0.8382" y="0.4318"/>
+<vertex x="-0.8382" y="64.8208"/>
+<vertex x="65.6844" y="64.8208"/>
 <vertex x="65.6844" y="0.4318"/>
 </polygon>
@@
 <wire x1="36.83" y1="33.274" x2="36.83" y2="34.29" width="0.3048" layer="1"/>
 <wire x1="36.83" y1="34.29" x2="38.354" y2="35.814" width="0.3048" layer="1"/>
-<wire x1="38.1" y1="7.6454" x2="27.94" y2="5.1054" width="0" layer="19" extent="1-1"/>
+<wire x1="20.8026" y1="41.1734" x2="16.764" y2="32.512" width="0" layer="19" extent="1-1"/>
+<wire x1="27.94" y1="5.1054" x2="38.1" y2="7.6454" width="0" layer="19" extent="1-1"/>
 </signal>
 <signal name="V_BAT">
@@
 <contactref element="U$1" pad="20-A6/TX5/LRCLK1"/>
 <wire x1="16.4592" y1="38.0492" x2="16.4592" y2="40.9448" width="0.3048" layer="16"/>
-<wire x1="16.4592" y1="40.9448" x2="13.208" y2="44.196" width="0.3048" layer="16"/>
-<wire x1="10.590021875" y1="44.196" x2="8.12916875" y2="46.656853125" width="0.3048" layer="16"/>
-<wire x1="13.208" y1="44.196" x2="10.590021875" y2="44.196" width="0.3048" layer="16"/>
+<wire x1="14.22516875" y1="46.910853125" x2="14.98716875" y2="46.148853125" width="0.3048" layer="16"/>
+<wire x1="14.98716875" y1="46.148853125" x2="14.98716875" y2="42.41683125" width="0.3048" layer="16"/>
+<wire x1="16.4592" y1="40.9448" x2="14.98716875" y2="42.41683125" width="0.3048" layer="16"/>
 </signal>
 <signal name="SERIAL_ESP_RX">
 <contactref element="JP3" pad="2"/>
 <contactref element="U$1" pad="21-A7/RX5/BCLK1"/>
-<wire x1="6.4964875" y1="44.7111" x2="6.5969" y2="44.7111" width="0.3048" layer="16"/>
-<wire x1="8.636" y1="42.672" x2="12.192" y2="42.672" width="0.3048" layer="16"/>
-<wire x1="12.192" y1="42.672" x2="13.9192" y2="40.9448" width="0.3048" layer="16"/>
+<wire x1="12.5924875" y1="44.9651" x2="13.3544875" y2="44.2031" width="0.3048" layer="16"/>
+<wire x1="13.3544875" y1="44.2031" x2="13.3544875" y2="41.5095125" width="0.3048" layer="16"/>
+<wire x1="13.3544875" y1="41.5095125" x2="13.9192" y2="40.9448" width="0.3048" layer="16"/>
 <wire x1="13.9192" y1="40.9448" x2="13.9192" y2="38.0492" width="0.3048" layer="16"/>
-<wire x1="6.5969" y1="44.7111" x2="8.636" y2="42.672" width="0.3048" layer="16"/>
 </signal>
 <signal name="SPI_CS">
@@
 </drawing>
 <compatibility>
+<note version="6.3" minversion="6.2.2" severity="warning">
+Since Version 6.2.2 text objects can contain more than one line,
+which will not be processed correctly with this version.
+</note>
 <note version="8.2" severity="warning">
 Since Version 8.2, EAGLE supports online libraries. The ids
