File: GMP_SCH.sch (EAGLE design)
At the start: 24 parts, among them CN1 1X4-3.5MM, CN2 1X4-3.5MM, IC1 MS560702BA03-50, Q1 TSM200N03DPQ33_RGG

Commit message: Add files via upload
V1.2, Test ready, Added decals
Connections:
- net GND renamed BARE
Changed lines of the file:
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@@
 </segment>
 </net>
-<net name="GND" class="0">
+<net name="BARE" class="0">
 <segment>
 <wire x1="-86.36" y1="196.85" x2="-88.9" y2="196.85" width="0.1524" layer="91"/>
